File: hardware/kicad/AD9364_IO.kicad_sch (KiCad schematic)
At the start: 7 parts, among them J5 Conn_Coaxial, U5 AD9364, Y2 X1E0000210808 40MHz

Commit message: update kicad files
Other:
- note added: "AD9364 IO"
- title: Murphy SDR -> MurPhy SDR
- moved on the sheet: R36, R37, U5G, U5H
