File: hardware/kicad/AD9364_RF.kicad_sch (KiCad schematic)
At the start: 41 parts, among them J3 Conn_Coaxial, J4 Conn_Coaxial, T1 TC1-1-13M+, T2 BD1631J50100AHF-CUSTOM, T3 TCM1-63AX+, U5 AD9364, U6 ADL5611

Commit message: update kicad files
Other:
- note added: "RF frontend"
- title: Murphy SDR -> MurPhy SDR
Changed lines of the file:
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@@
 	(paper "A3")
 	(title_block
-		(title "Murphy SDR")
+		(title "MurPhy SDR")
 		(date "2024-04-22")
 		(company "M.P Inc")
