File: hardware/kicad/AD9364_power-supply.kicad_sch (KiCad schematic)
At the start: 30 parts, among them U5 AD9364

Commit message: update kicad files
Other:
- note added: "AD9364 power"
- title: Murphy SDR -> MurPhy SDR
Changed lines of the file:
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@@
 	(paper "A4")
 	(title_block
-		(title "Murphy SDR")
+		(title "MurPhy SDR")
 		(date "2024-04-22")
 		(company "M.P Inc")
