File: hardware/kicad/FT601Q.kicad_sch (KiCad schematic)
At the start: 39 parts, among them J2 USB3_A, U3 ESD7016, U4 FT601Q, Y1 30MHz crystal

Commit message: update kicad files
Other:
- note added: "FT601Q USB 3.0 interface"
- title: Murphy SDR -> MurPhy SDR
Changed lines of the file:
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@@
 	(paper "A3")
 	(title_block
-		(title "Murphy SDR")
+		(title "MurPhy SDR")
 		(date "2024-04-22")
 		(company "M.P Inc")
