File: hardware/kicad/MurPhySDR.kicad_sch (KiCad schematic)
At the start: 4 parts

Commit message: update kicad files
Other:
- note added: "FPGA XC7A50T-2FTGI"
- note added: "MurPhy SDR"
- note added: "Transceiver AD9364"
- note added: "USB interface FT601Q"
- title: Murphy SDR -> MurPhy SDR
- moved on the sheet: H1, H2, H3, H4
