File: hardware/kicad/Xilinx_Artix-7_Banks.kicad_sch (KiCad schematic)
At the start: 17 parts, among them J1 878321420, U1 XC7A50T-2FTG256I, U2 MX25L25645GZNI-08G-CUSTOM

Commit message: update kicad files
Other:
- note added: "FPGA banks, JTAG and FLASH"
- note added: "JTAG"
- note removed: "1.8V for AD9364!!!"
- note removed: "3.3V for FTDI!!!"
- title: Murphy SDR -> MurPhy SDR
Changed lines of the file:
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@@
 	(paper "A3")
 	(title_block
-		(title "Murphy SDR")
+		(title "MurPhy SDR")
 		(date "2024-04-22")
 		(company "M.P Inc")
@@
 	)
 	(rectangle
+		(start 254 186.69)
+		(end 270.51 194.31)
+		(stroke
+			(width 0.2159)
+			(type default)
+		)
+		(fill
+			(type none)
+		)
+	)
+	(rectangle
 		(start 34.29 24.13)
 		(end 73.66 31.75)
 		(stroke
-			(width 0.15)
+			(width 0.2159)
 			(type default)
 		)
@@
 		)
 	)
-	(text "1.8V for AD9364!!!"
+	(text "FPGA banks, JTAG and FLASH"
 		(exclude_from_sim no)
-		(at 306.07 261.62 0)
+		(at 334.264 256.794 0)
 		(effects
 			(font
-				(size 2 2)
+				(face "DejaVu Serif")
+				(size 2.794 2.794)
+				(thickness 1.016)
+				(bold yes)
+				(italic yes)
+				(color 0 0 0 1)
 			)
-			(justify left bottom)
 		)
 	)
-	(text "3.3V for FTDI!!!"
+	(text "JTAG"
 		(exclude_from_sim no)
-		(at 305.816 265.938 0)
+		(at 255.27 193.04 0)
 		(effects
 			(font
-				(size 2 2)
+				(face "KiCad Font")
+				(size 4 4)
 			)
 			(justify left bottom)
