File: hardware/kicad/Xilinx_Artix-7_power-supply.kicad_sch (KiCad schematic)
At the start: 44 parts, among them U1 XC7A50T-2FTG256I

Commit message: update kicad files
Other:
- note added: "FPGA power"
- title: Murphy SDR -> MurPhy SDR
Changed lines of the file:
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@@
 	(paper "A3")
 	(title_block
-		(title "Murphy SDR")
+		(title "MurPhy SDR")
 		(date "2024-04-22")
 		(company "M.P Inc")
@@
 		)
 	)
+	(text "FPGA power"
+		(exclude_from_sim no)
+		(at 314.706 256.794 0)
+		(effects
+			(font
+				(face "DejaVu Serif")
+				(size 2.794 2.794)
+				(thickness 1.016)
+				(bold yes)
+				(italic yes)
+				(color 0 0 0 1)
+			)
+		)
+	)
