File: hardware/kicad/power-supply.kicad_sch (KiCad schematic)
At the start: 41 parts, among them IC1 LMZ30604RKGT, IC2 LMZ30604RKGT, IC3 LMZ30604RKGT, IC4 ADP1755ACPZ-R7, IC5 ADP1755ACPZ-R7

Commit message: update kicad files
Other:
- note added: "Power supply"
- title: Murphy SDR -> MurPhy SDR
Changed lines of the file:
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@@
 	(paper "A3")
 	(title_block
-		(title "Murphy SDR")
+		(title "MurPhy SDR")
 		(date "2024-04-22")
 		(company "M.P Inc")
